Commit message: Primera versao garra do robo

File: description/robot.urdf.xacro (robot description, xacro)
@@ -209,43 +209,59 @@
     <origin xyz="0 0 0.01"/>
   </joint>
-<!-- Define um sistema de controle ROS 2 utilizando a infraestrutura ros2_control -->
-<ros2_control name="IgnitionSystem" type="system">
-  <!-- Seção de hardware do sistema, onde é especificado o plugin que fará a ponte entre o Gazebo (Ignition) e o ros2_control -->
-  <hardware>
-    <!-- Plugin que permite a integração entre o Ignition Gazebo e o framework ros2_control -->
-    <plugin>ign_ros2_control/IgnitionSystem</plugin>
-  </hardware>
-  <!-- Definição do primeiro atuador, correspondente à roda esquerda ("drive wheel left") -->
-  <joint name="drivewhl_l_joint">
-    <!-- Interface de comando de velocidade angular (por exemplo, rad/s) para essa junta -->
-    <command_interface name="velocity">
-      <!-- Valor mínimo permitido para o comando de velocidade (limite inferior) -->
-      <param name="min">-1</param>
-      <!-- Valor máximo permitido para o comando de velocidade (limite superior) -->
-      <param name="max">1</param>
-    </command_interface>
-    <!-- Interface de estado que fornece a posição atual da junta (por exemplo, em radianos) -->
-    <state_interface name="position"/>
-    <!-- Interface de estado que fornece a velocidade atual da junta (por exemplo, em rad/s) -->
-    <state_interface name="velocity"/>
-  </joint>
-  <!-- Definição do segundo atuador, correspondente à roda direita ("drive wheel right") -->
-  <joint name="drivewhl_r_joint">
-    <!-- Interface de comando de velocidade angular para essa junta -->
-    <command_interface name="velocity">
-      <!-- Limite inferior da velocidade que pode ser comandada -->
-      <param name="min">-1</param>
-      <!-- Limite superior da velocidade que pode ser comandada -->
-      <param name="max">1</param>
-    </command_interface>
-    <!-- Interface de estado para leitura da posição da junta -->
-    <state_interface name="position"/>
-    <!-- Interface de estado para leitura da velocidade da junta -->
-    <state_interface name="velocity"/>
-  </joint>
-</ros2_control>
+  <!-- Define um sistema de controle ROS 2 utilizando a infraestrutura ros2_control -->
+  <ros2_control name="IgnitionSystem" type="system">
+    <!-- Seção de hardware do sistema, onde é especificado o plugin que fará a ponte entre o Gazebo (Ignition) e o ros2_control -->
+    <hardware>
+      <!-- Plugin que permite a integração entre o Ignition Gazebo e o framework ros2_control -->
+      <plugin>ign_ros2_control/IgnitionSystem</plugin>
+    </hardware>
+    <!-- Definição do primeiro atuador, correspondente à roda esquerda ("drive wheel left") -->
+    <joint name="drivewhl_l_joint">
+      <!-- Interface de comando de velocidade angular (por exemplo, rad/s) para essa junta -->
+      <command_interface name="velocity">
+        <!-- Valor mínimo permitido para o comando de velocidade (limite inferior) -->
+        <param name="min">-1</param>
+        <!-- Valor máximo permitido para o comando de velocidade (limite superior) -->
+        <param name="max">1</param>
+      </command_interface>
+      <!-- Interface de estado que fornece a posição atual da junta (por exemplo, em radianos) -->
+      <state_interface name="position"/>
+      <!-- Interface de estado que fornece a velocidade atual da junta (por exemplo, em rad/s) -->
+      <state_interface name="velocity"/>
+    </joint>
+    <!-- Definição do segundo atuador, correspondente à roda direita ("drive wheel right") -->
+    <joint name="drivewhl_r_joint">
+      <!-- Interface de comando de velocidade angular para essa junta -->
+      <command_interface name="velocity">
+        <!-- Limite inferior da velocidade que pode ser comandada -->
+        <param name="min">-1</param>
+        <!-- Limite superior da velocidade que pode ser comandada -->
+        <param name="max">1</param>
+      </command_interface>
+      <!-- Interface de estado para leitura da posição da junta -->
+      <state_interface name="position"/>
+      <!-- Interface de estado para leitura da velocidade da junta -->
+      <state_interface name="velocity"/>
+    </joint>
+    <joint name="gripper_extension">
+      <command_interface name="position">
+        <param name="min">-1.57075</param>
+        <param name="max">0.0</param>
+      </command_interface>
+      <state_interface name="position"/>
+      <state_interface name="velocity"/>
+    </joint>
+    <joint name="right_gripper_joint">
+      <command_interface name="position">
+        <param name="min">-0.38</param>
+        <param name="max">0.0</param>
+      </command_interface>
+      <state_interface name="position"/>
+      <state_interface name="velocity"/>
+    </joint>
+  </ros2_control>
   <gazebo>
     <plugin filename="ign_ros2_control-system" name="ign_ros2_control::IgnitionROS2ControlPlugin">
-      <parameters>$(find prm)/config/diff_drive_controller_velocity.yaml</parameters>
+      <parameters>$(find prm)/config/controller_config.yaml</parameters>
     </plugin>
   </gazebo>
@@ -445,3 +461,75 @@
     </sensor> -->
   </gazebo>
+  <joint name="gripper_extension" type="revolute">
+    <axis xyz="0 1 0"/>
+    <limit effort="5000.0" lower="-1.57075" upper="0.0" velocity="0.5"/>
+    <origin rpy="0 0 0" xyz="0.19 0 0.1"/>
+    <parent link="base_link"/>
+    <child link="gripper_pole"/>
+  </joint>
+  <link name="gripper_pole">
+    <visual>
+      <geometry>
+        <cylinder length="0.2" radius="0.01"/>
+      </geometry>
+      <origin rpy="0 1.57075 0" xyz="0.1 0 0"/>
+    </visual>
+    <xacro:cylinder_inertia m="0.01" r="0.01" h="0.2"/>
+  </link>
+  <joint name="left_gripper_joint" type="fixed">
+    <origin rpy="0 0 0" xyz="0.2 0.01 0"/>
+    <parent link="gripper_pole"/>
+    <child link="left_gripper"/>
+  </joint>
+  <link name="left_gripper">
+    <visual>
+      <origin rpy="0.0 0 0" xyz="0 0 0"/>
+      <geometry>
+        <box size="0.1 0.02 0.02"/> <!-- Comprimento, largura, altura -->
+      </geometry>
+    </visual>
+    <xacro:box_inertia m="0.015" w="0.02" h="0.02" d="0.1"/>
+  </link>
+  <joint name="left_tip_joint" type="fixed">
+    <parent link="left_gripper"/>
+    <child link="left_tip"/>
+  </joint>
+  <link name="left_tip">
+    <visual>
+      <origin rpy="0.0 0 0" xyz="0.09137 0.00495 0"/>
+      <geometry>
+        <box size="0.02 0.01 0.01"/>
+      </geometry>
+    </visual>
+    <xacro:box_inertia m="0.005" w="0.01" h="0.01" d="0.02"/>
+  </link>
+  <joint name="right_gripper_joint" type="prismatic">
+    <axis xyz="0 1 0"/>
+    <limit effort="1000.0" lower="-0.38" upper="0" velocity="0.5"/>
+    <origin rpy="0 0 0" xyz="0.2 -0.01 0"/>
+    <parent link="gripper_pole"/>
+    <child link="right_gripper"/>
+  </joint>
+  <link name="right_gripper">
+    <visual>
+      <origin rpy="-3.1415 0 0" xyz="0 0 0"/>
+      <geometry>
+        <box size="0.1 0.02 0.02"/>
+      </geometry>
+    </visual>
+    <xacro:box_inertia m="0.015" w="0.02" h="0.02" d="0.1"/>
+  </link>
+  <joint name="right_tip_joint" type="fixed">
+    <parent link="right_gripper"/>
+    <child link="right_tip"/>
+  </joint>
+  <link name="right_tip">
+    <visual>
+      <origin rpy="-3.1415 0 0" xyz="0.09137 0.00495 0"/>
+      <geometry>
+        <box size="0.02 0.01 0.01"/>
+      </geometry>
+    </visual>
+    <xacro:box_inertia m="0.005" w="0.01" h="0.01" d="0.02"/>
+  </link>
 </robot>

Commit message: Correcao de constantes fisicas da garra, melhoria do seu posicionamento, correcao de problemas com o teste_urdf.launch.py

File: description/robot.urdf.xacro (robot description, xacro)
@@ -247,5 +247,13 @@
       <command_interface name="position">
         <param name="min">-1.57075</param>
-        <param name="max">0.0</param>
+        <param name="max">0.2</param>
+      </command_interface>
+      <state_interface name="position"/>
+      <state_interface name="velocity"/>
+    </joint>
+    <joint name="left_gripper_joint">
+      <command_interface name="position">
+        <param name="min">0.0</param>
+        <param name="max">0.06</param>
       </command_interface>
       <state_interface name="position"/>
@@ -254,5 +262,5 @@
     <joint name="right_gripper_joint">
       <command_interface name="position">
-        <param name="min">-0.38</param>
+        <param name="min">-0.06</param>
         <param name="max">0.0</param>
       </command_interface>
@@ -463,6 +471,6 @@
   <joint name="gripper_extension" type="revolute">
     <axis xyz="0 1 0"/>
-    <limit effort="5000.0" lower="-1.57075" upper="0.0" velocity="0.5"/>
-    <origin rpy="0 0 0" xyz="0.19 0 0.1"/>
+    <limit effort="50.0" lower="-1.57075" upper="0.2" velocity="0.5"/>
+    <origin rpy="0 0 0" xyz="0.2 0 0.1"/>
     <parent link="base_link"/>
     <child link="gripper_pole"/>
@@ -475,7 +483,14 @@
       <origin rpy="0 1.57075 0" xyz="0.1 0 0"/>
     </visual>
+    <collision>
+      <geometry>
+        <cylinder length="0.2" radius="0.01"/>
+      </geometry>
+    </collision>
     <xacro:cylinder_inertia m="0.01" r="0.01" h="0.2"/>
   </link>
-  <joint name="left_gripper_joint" type="fixed">
+  <joint name="left_gripper_joint" type="prismatic">
+    <axis xyz="0 1 0"/>
+    <limit effort="100.0" lower="0.0" upper="0.06" velocity="0.25"/>
     <origin rpy="0 0 0" xyz="0.2 0.01 0"/>
     <parent link="gripper_pole"/>
@@ -484,12 +499,17 @@
   <link name="left_gripper">
     <visual>
-      <origin rpy="0.0 0 0" xyz="0 0 0"/>
       <geometry>
         <box size="0.1 0.02 0.02"/> <!-- Comprimento, largura, altura -->
       </geometry>
     </visual>
+    <collision>
+      <geometry>
+        <box size="0.1 0.02 0.02"/>
+      </geometry>
+    </collision>
     <xacro:box_inertia m="0.015" w="0.02" h="0.02" d="0.1"/>
   </link>
   <joint name="left_tip_joint" type="fixed">
+    <origin rpy="0.0 0 0" xyz="0.06 0.001 0"/>
     <parent link="left_gripper"/>
     <child link="left_tip"/>
@@ -497,14 +517,20 @@
   <link name="left_tip">
     <visual>
-      <origin rpy="0.0 0 0" xyz="0.09137 0.00495 0"/>
-      <geometry>
-        <box size="0.02 0.01 0.01"/>
-      </geometry>
-    </visual>
-    <xacro:box_inertia m="0.005" w="0.01" h="0.01" d="0.02"/>
+      <origin rpy="0 0 -0.1" xyz="0.03 0 0"/>
+      <geometry>
+        <box size="0.06 0.01 0.01"/>
+      </geometry>
+    </visual>
+    <collision>
+      <origin rpy="0 0 -0.1" xyz="0.03 0 0"/>
+      <geometry>
+        <box size="0.06 0.01 0.01"/>
+      </geometry>
+    </collision>
+    <xacro:box_inertia m="0.005" w="0.01" h="0.01" d="0.06"/>
   </link>
   <joint name="right_gripper_joint" type="prismatic">
     <axis xyz="0 1 0"/>
-    <limit effort="1000.0" lower="-0.38" upper="0" velocity="0.5"/>
+    <limit effort="100.0" lower="-0.06" upper="0" velocity="0.25"/>
     <origin rpy="0 0 0" xyz="0.2 -0.01 0"/>
     <parent link="gripper_pole"/>
@@ -518,7 +544,14 @@
       </geometry>
     </visual>
+    <collision>
+      <origin rpy="-3.1415 0 0" xyz="0 0 0"/>
+      <geometry>
+        <box size="0.1 0.02 0.02"/>
+      </geometry>
+    </collision>
     <xacro:box_inertia m="0.015" w="0.02" h="0.02" d="0.1"/>
   </link>
   <joint name="right_tip_joint" type="fixed">
+    <origin rpy="-3.1415 0 0" xyz="0.06 -0.001 0"/>
     <parent link="right_gripper"/>
     <child link="right_tip"/>
@@ -526,10 +559,16 @@
   <link name="right_tip">
     <visual>
-      <origin rpy="-3.1415 0 0" xyz="0.09137 0.00495 0"/>
-      <geometry>
-        <box size="0.02 0.01 0.01"/>
-      </geometry>
-    </visual>
-    <xacro:box_inertia m="0.005" w="0.01" h="0.01" d="0.02"/>
+      <origin rpy="0 0 -0.1" xyz="0.03 0 0"/>
+      <geometry>
+        <box size="0.06 0.01 0.01"/>
+      </geometry>
+    </visual>
+    <collision>
+      <origin rpy="0 0 -0.1" xyz="0.03 0 0"/>
+      <geometry>
+        <box size="0.06 0.01 0.01"/>
+      </geometry>
+    </collision>
+    <xacro:box_inertia m="0.005" w="0.01" h="0.01" d="0.06"/>
   </link>
 </robot>

File: world/empty_arena.sdf.xacro (robot description, xacro)
@@ -2,5 +2,5 @@
 <robot xmlns:xacro="http://www.ros.org/wiki/xacro" name="capture_the_flag_world">
     <!-- Gerando o SDF:
-        $ xacro empty_arena.sdf.xacro. > arena_2.sdf
+        $ xacro empty_arena.sdf.xacro > empty_arena.sdf
      -->
     <!-- Parâmetros globais -->
@@ -30,6 +30,6 @@
     <xacro:property name="flag_panel_size"   value="0.3 0.01 0.2"/>
     <xacro:property name="flag_panel_pose"   value="0.16 0 0.38 0 0 0"/>
-    <xacro:property name="flag_collision_pose" value="0.08 0 0.2 0 0 0"/>
-    <xacro:property name="flag_collision_size" value="0.15 0.15 0.4"/>
+    <xacro:property name="flag_base_radius" value="0.05"/>
+    <xacro:property name="flag_base_thickness" value="0.01"/>
     <xacro:macro name="bandeira" params="name x y z rot cor label">
         <model name="${name}">
@@ -69,9 +69,40 @@
                 <!-- Colisão -->
                 <collision name="${name}_collision">
-                    <pose>${flag_collision_pose}</pose>
+                    <pose>0 0 ${flag_pole_length/2} 0 0 0</pose>
                     <geometry>
                     <box>
-                        <size>${flag_collision_size}</size>
+                        <size>${flag_pole_radius*2} ${flag_pole_radius*2} ${flag_pole_length} </size>
                     </box>
+                    </geometry>
+                </collision>
+                <!-- Base da bandeira (visual) -->
+                <visual name="base_visual">
+                    <pose>0 0 ${flag_base_thickness/2} 0 0 0</pose>
+                    <geometry>
+                        <cylinder>
+                        <radius>${flag_base_radius}</radius>
+                        <length>${flag_base_thickness}</length>
+                        </cylinder>
+                    </geometry>
+                    <material>
+                        <ambient>0.1 0.1 0.1 1</ambient>
+                        <diffuse>0.2 0.2 0.2 1</diffuse>
+                    </material>
+                </visual>
+                <!-- Base da bandeira (colisão) -->
+                <collision name="base_collision">
+                    <pose>0 0 ${flag_base_thickness/2} 0 0 0</pose>
+                    <geometry>
+                        <box>
+                            <size>${flag_base_radius*2} ${flag_base_radius*2} ${flag_base_thickness} </size>
+                        </box>
+                    </geometry>
+                </collision>
+                <collision name="top_base_collision">
+                    <pose>0 0 ${flag_pole_length*0.75} 0 0 0</pose>
+                    <geometry>
+                        <box>
+                            <size>${flag_base_radius*2} ${flag_base_radius*2} ${flag_base_thickness} </size>
+                        </box>
                     </geometry>
                 </collision>
